Commit message: Updated bigman and coman models; now using ACM from SRDF

File: tests/robots/bigman/bigman.urdf (robot description, URDF)
Before this commit: robot bigman, 76 links, 75 joints
Links:
- removed link l_hand_lower_left_link
- removed link l_hand_lower_right_link
- removed link l_hand_upper_left_link
- removed link l_hand_upper_right_link
- removed link r_hand_lower_left_link
- removed link r_hand_lower_right_link
- removed link r_hand_upper_left_link
- removed link r_hand_upper_right_link
- added link LRaisingSupport, mass 1.3789343; collision box size=0.218 0.04 0.152; visual mesh filename=package://bigman_urdf/meshes/RaisingSupport.STL scale=0.001 -0.001 0.001
- added link LSoftHandLink, mass 5.0e-01; collision mesh filename=package://bigman_urdf/meshes/simple/SoftHandOpen.STL scale=0.001 -0.001 0.001; visual mesh filename=package://bigman_urdf/meshes/SoftHandOpen.STL scale=0.001 -0.001 0.001
- added link NeckPitch, mass 1.0; collision mesh filename=package://bigman_urdf/meshes/simple/NeckPitch.STL scale=0.001 0.001 0.001; visual mesh filename=package://bigman_urdf/meshes/NeckPitch.STL scale=0.001 0.001 0.001
- added link NeckYaw, mass 1.0; collision mesh filename=package://bigman_urdf/meshes/simple/NeckYaw.STL scale=0.001 0.001 0.001; visual mesh filename=package://bigman_urdf/meshes/NeckYaw.STL scale=0.001 0.001 0.001
- added link RRaisingSupport, mass 1.3789343; collision box size=0.218 0.04 0.152; visual mesh filename=package://bigman_urdf/meshes/RaisingSupport.STL scale=0.001 0.001 0.001
- added link RSoftHandLink, mass 5.0e-01; collision mesh filename=package://bigman_urdf/meshes/simple/SoftHandOpen.STL scale=0.001 0.001 0.001; visual mesh filename=package://bigman_urdf/meshes/SoftHandOpen.STL scale=0.001 0.001 0.001
- added link l_forearm_backward_contact_link
- added link l_forearm_central_contact_link
- added link l_forearm_forward_contact_link
- added link l_palm
- added link r_forearm_backward_contact_link
- added link r_forearm_central_contact_link
- added link r_forearm_forward_contact_link
- added link r_palm
- link DWYTorso: geometry collision mesh filename=package://bigman_urdf/meshes/simple/NewChest.STL scale=0.001 0.001 0.001; visual mesh filename=package://bigman_urdf/meshes/NewChest.STL scale=0.001 0.001 0.001
- link LFoot: geometry collision box size=0.306 0.16 0.015; visual mesh filename=package://bigman_urdf/meshes/Foot.STL scale=0.001 0.001 0.001
- link LLowLeg: geometry collision mesh filename=package://bigman_urdf/meshes/simple/KneePitchCalf.STL scale=0.001 -0.001 0.001; visual mesh filename=package://bigman_urdf/meshes/KneePitchCalf.STL scale=0.001 -0.001 0.001
- link LSoftHand: mass 0.3 -> None; geometry 
- link RFoot: geometry collision box size=0.306 0.16 0.015; visual mesh filename=package://bigman_urdf/meshes/Foot.STL scale=0.001 -0.001 0.001
- link RLowLeg: geometry collision mesh filename=package://bigman_urdf/meshes/simple/KneePitchCalf.STL scale=0.001 0.001 0.001; visual mesh filename=package://bigman_urdf/meshes/KneePitchCalf.STL scale=0.001 0.001 0.001
- link RSoftHand: mass 0.3 -> None; geometry 
- link center_bottom_led_frame: mass 1e-5 -> None
- link center_top_led_frame: mass 1e-5 -> None
- link head: geometry collision mesh filename=package://bigman_urdf/meshes/simple/Head.STL scale=0.001 0.001 0.001; visual mesh filename=package://bigman_urdf/meshes/Head.STL scale=0.001 0.001 0.001
- link head_hokuyo_frame: mass 1e-5 -> None
- link left_camera_frame: mass 1e-5 -> None
- link left_led_frame: mass 1e-5 -> None
- link right_camera_frame: mass 1e-5 -> None
- link right_led_frame: mass 1e-5 -> None
Joints:
- removed joint l_hand_lower_left_joint
- removed joint l_hand_lower_right_joint
- removed joint l_hand_upper_left_joint
- removed joint l_hand_upper_right_joint
- removed joint r_hand_lower_left_joint
- removed joint r_hand_lower_right_joint
- removed joint r_hand_upper_left_joint
- removed joint r_hand_upper_right_joint
- added joint LRaisingSupport_joint: type fixed, parent LWrMot2, child LRaisingSupport, origin xyz=0.0 0.0 -0.0505 rpy=0 0 0
- added joint NeckPitchj: type revolute, parent NeckYaw, child NeckPitch, origin xyz=0 0 0.1155 rpy=0 0 0, axis 0 1 0, limit lower=-0.523598775597 upper=1.22173047639 effort=120 velocity=6.283
- added joint NeckYawj: type revolute, parent DWYTorso, child NeckYaw, origin xyz=0 0 0 rpy=0 0 0, axis 0 0 1, limit lower=-3.05432619098 upper=3.05432619098 effort=120 velocity=6.283
- added joint RRaisingSupport_joint: type fixed, parent RWrMot2, child RRaisingSupport, origin xyz=0.0 0.0 -0.0505 rpy=0 0 0
- added joint l_forearm_backward_contact_joint: type fixed, parent LRaisingSupport, child l_forearm_backward_contact_link, origin xyz=-0.081 0 -0.132 rpy=0 0 0
- added joint l_forearm_central_contact_joint: type fixed, parent LRaisingSupport, child l_forearm_central_contact_link, origin xyz=0.0 0 -0.152 rpy=0 0 0
- added joint l_forearm_forward_contact_joint: type fixed, parent LRaisingSupport, child l_forearm_forward_contact_link, origin xyz=0.097 0 -0.132 rpy=0 0 0
- added joint l_handj2: type fixed, parent LSoftHandLink, child LSoftHand, origin xyz=0.011908576 -0.0021833446 -0.15361558 rpy=0 0 0
- added joint l_handj3: type fixed, parent LSoftHand, child l_palm, origin xyz=0 -0.025696923 0.0 rpy=0 0 0
- added joint r_forearm_backward_contact_joint: type fixed, parent RRaisingSupport, child r_forearm_backward_contact_link, origin xyz=-0.081 0 -0.132 rpy=0 0 0
- added joint r_forearm_central_contact_joint: type fixed, parent RRaisingSupport, child r_forearm_central_contact_link, origin xyz=0.0 0 -0.152 rpy=0 0 0
- added joint r_forearm_forward_contact_joint: type fixed, parent RRaisingSupport, child r_forearm_forward_contact_link, origin xyz=0.097 0 -0.132 rpy=0 0 0
- added joint r_handj2: type fixed, parent RSoftHandLink, child RSoftHand, origin xyz=0.011908576 0.0021833446 -0.15361558 rpy=0 0 0
- added joint r_handj3: type fixed, parent RSoftHand, child r_palm, origin xyz=0 0.025696923 0.0 rpy=0 0 0
- joint LElbj: limit lower=-2.966 upper=0.523 effort=60 velocity=6.283 -> lower=-2.96705972838 upper=0.593411945677 effort=60 velocity=6.283
- joint LShLat: limit lower=0.052 upper=3.699 effort=120 velocity=6.283 -> lower=0.0872664625995 upper=3.8571776469 effort=120 velocity=6.283
- joint LShSag: axis 0 0.743144825 0.669130606 -> 0.0 0.743144825 0.669130606; limit lower=-2.844 upper=2.844 effort=120 velocity=6.283 -> lower=-2.87979326578 upper=2.79252680318 effort=120 velocity=6.283; origin xyz=0.0 0.2 0.0 rpy=0 0 0 -> xyz=0.045646 0.219164 0.001531 rpy=0 0 -0.3491
- joint LShYaw: limit lower=-2.844 upper=2.844 effort=120 velocity=6.283 -> lower=-2.84488668074 upper=2.84488668074 effort=120 velocity=6.283
- joint RElbj: limit lower=-2.966 upper=0.523 effort=60 velocity=6.283 -> lower=-2.96705972838 upper=0.593411945677 effort=60 velocity=6.283
- joint RShLat: limit lower=-3.699 upper=-0.052 effort=120 velocity=6.283 -> lower=-3.8571776469 upper=-0.122173047639 effort=120 velocity=6.283
- joint RShSag: limit lower=-2.844 upper=2.844 effort=120 velocity=6.283 -> lower=-2.84488668074 upper=2.8099800957 effort=120 velocity=6.283; origin xyz=0.0 -0.2 0.0 rpy=0 0 0 -> xyz=0.045646 -0.219164 0.001531 rpy=0 0 0.3491
- joint RShYaw: limit lower=-2.844 upper=2.844 effort=120 velocity=6.283 -> lower=-2.86233997326 upper=2.82743338822 effort=120 velocity=6.283
- joint WaistLat: limit lower=-0.610 upper=0.610 effort=120 velocity=6.283 -> lower=-0.610865238196 upper=0.610865238196 effort=120 velocity=6.283
- joint WaistSag: limit lower=-0.349 upper=1.396 effort=220 velocity=6.283 -> lower=-0.349065850398 upper=1.39626340159 effort=220 velocity=6.283
- joint WaistYaw: limit lower=-2.844 upper=2.844 effort=120 velocity=6.283 -> lower=-2.09439510239 upper=2.09439510239 effort=120 velocity=6.283
- joint gaze_joint: origin xyz=0 0 0.1 rpy=0 0 0 -> xyz=0 0 0 rpy=0 0 0; parent torso -> head
- joint imu_joint: origin xyz=-0.072 -0.0068 0.044 rpy=0 3.14159265359 0 -> xyz=-0.072 -0.0068 0.044 rpy=0 0 0
- joint l_foot_lower_left_joint: origin xyz=-0.111 0.07 0 rpy=0 0 0 -> xyz=-0.111 0.09 0 rpy=0 0 0
- joint l_foot_lower_right_joint: origin xyz=-0.111 -0.09 0 rpy=0 0 0 -> xyz=-0.111 -0.07 0 rpy=0 0 0
- joint l_foot_upper_left_joint: origin xyz=0.195 0.07 0 rpy=0 0 0 -> xyz=0.195 0.09 0 rpy=0 0 0
- joint l_foot_upper_right_joint: origin xyz=0.195 -0.09 0 rpy=0 0 0 -> xyz=0.195 -0.07 0 rpy=0 0 0
- joint l_handj: child LSoftHand -> LSoftHandLink; origin xyz=0 0 -0.11 rpy=0 0 0 -> xyz=0 0 0 rpy=0 0 0
- joint l_leg_ft_joint: parent LFootmot -> LFoot
- joint left_led_frame_joint: origin xyz=-0.01443 0.07452 0.050346 rpy=0 -0.15 0.53 -> xyz=-0.01443 0.07452 0.050346 rpy=0 0 0.6
- joint neck_joint: origin xyz=0.05 0 0.05 rpy=0 0 0 -> xyz=0.08765 0 0.06475 rpy=0 0 0; parent DWYTorso -> NeckPitch
- joint r_foot_lower_left_joint: origin xyz=-0.111 -0.07 0 rpy=0 0 0 -> xyz=-0.111 -0.09 0 rpy=0 0 0
- joint r_foot_lower_right_joint: origin xyz=-0.111 0.09 0 rpy=0 0 0 -> xyz=-0.111 0.07 0 rpy=0 0 0
- joint r_foot_upper_left_joint: origin xyz=0.195 -0.07 0 rpy=0 0 0 -> xyz=0.195 -0.09 0 rpy=0 0 0
- joint r_foot_upper_right_joint: origin xyz=0.195 0.09 0 rpy=0 0 0 -> xyz=0.195 0.07 0 rpy=0 0 0
- joint r_handj: child RSoftHand -> RSoftHandLink; origin xyz=0 0 -0.11 rpy=0 0 0 -> xyz=0 0 0 rpy=0 0 0
- joint r_leg_ft_joint: parent RFootmot -> RFoot
- joint right_led_frame_joint: origin xyz=-0.01443 -0.07452 0.050346 rpy=0 -0.15 -0.53 -> xyz=-0.01443 -0.07452 0.050346 rpy=0 0 -0.6

Commit message: Fixed compilation issues for collision_utils. Added a function to update iDyn3 from a joint state msg. Added a capsule version of bigman. Added an example for collision_utils where a number of minimum distance points is published

File: tests/robots/bigman/bigman.urdf (robot description, URDF)
Before this commit: robot bigman, 82 links, 81 joints
Links:
- removed link LRaisingSupport
- removed link RRaisingSupport
- removed link center_bottom_led_frame
- removed link center_top_led_frame
- removed link head
- removed link head_hokuyo_frame
- removed link head_imu_link
- removed link hokuyo_link
- removed link l_forearm_backward_contact_link
- removed link l_forearm_central_contact_link
- removed link l_forearm_forward_contact_link
- removed link l_palm
- removed link left_camera_frame
- removed link left_camera_optical_frame
- removed link left_led_frame
- removed link r_forearm_backward_contact_link
- removed link r_forearm_central_contact_link
- removed link r_forearm_forward_contact_link
- removed link r_palm
- removed link right_camera_frame
- removed link right_camera_optical_frame
- removed link right_led_frame
- added link TorsoProtections, mass 4.7; collision mesh filename=package://bigman_urdf/meshes/simple/ProtectionSystem.STL scale=0.001 0.001 0.001; visual mesh filename=package://bigman_urdf/meshes/ProtectionSystem.STL scale=0.001 0.001 0.001
- added link backpack, mass 10.0; collision box size=0.16 0.3 0.22; visual box size=0.16 0.3 0.22
- added link multisense/center_bottom_led_frame
- added link multisense/center_top_led_frame
- added link multisense/head, mass 1.41984; collision mesh filename=package://bigman_urdf/meshes/simple/Head.STL scale=0.001 0.001 0.001; visual mesh filename=package://bigman_urdf/meshes/Head.STL scale=0.001 0.001 0.001
- added link multisense/head_hokuyo_frame
- added link multisense/head_imu_link, mass 1e-5; visual box size=0.01 0.01 0.01
- added link multisense/hokuyo_link, mass 0.057654; collision box size=0.08 0.06 0.04238; collision cylinder length=0.047 radius=0.024425
- added link multisense/left_camera_frame
- added link multisense/left_camera_optical_frame
- added link multisense/left_led_frame
- added link multisense/right_camera_frame
- added link multisense/right_camera_optical_frame
- added link multisense/right_led_frame
- link DWYTorso: mass 22.38913469 -> 7.31313212
- link LSoftHandLink: mass 5.0e-01 -> 1.2
- link NeckPitch: mass 1.0 -> 0.623
- link NeckYaw: mass 1.0 -> 0.35
- link RSoftHandLink: mass 5.0e-01 -> 1.2
- link Waist: mass 6.4080904 -> 1.1046081e+01
Joints:
- removed joint LRaisingSupport_joint
- removed joint RRaisingSupport_joint
- removed joint l_forearm_backward_contact_joint
- removed joint l_forearm_central_contact_joint
- removed joint l_forearm_forward_contact_joint
- removed joint l_handj3
- removed joint r_forearm_backward_contact_joint
- removed joint r_forearm_central_contact_joint
- removed joint r_forearm_forward_contact_joint
- removed joint r_handj3
- added joint backpack_joint: type fixed, parent DWYTorso, child backpack, origin xyz=-0.185 0 -0.025 rpy=0 0 0
- added joint torso_protection_joint: type fixed, parent DWYTorso, child TorsoProtections, origin xyz=0.0 0 0.0 rpy=0 0 0
- joint LShLat: limit lower=0.0872664625995 upper=3.8571776469 effort=120 velocity=6.283 -> lower=0.0872664625995 upper=2.96705972838 effort=120 velocity=6.283
- joint LShSag: limit lower=-2.87979326578 upper=2.79252680318 effort=120 velocity=6.283 -> lower=-0.994837673634 upper=1.55334303427 effort=120 velocity=6.283
- joint NeckPitchj: limit lower=-0.523598775597 upper=1.22173047639 effort=120 velocity=6.283 -> lower=-0.436332312998 upper=1.04719755119 effort=120 velocity=6.283
- joint RShLat: limit lower=-3.8571776469 upper=-0.122173047639 effort=120 velocity=6.283 -> lower=-2.96705972838 upper=-0.122173047639 effort=120 velocity=6.283
- joint RShSag: limit lower=-2.84488668074 upper=2.8099800957 effort=120 velocity=6.283 -> lower=-0.994837673634 upper=1.55334303427 effort=120 velocity=6.283
- joint WaistLat: limit lower=-0.610865238196 upper=0.610865238196 effort=120 velocity=6.283 -> lower=-0.261799387798 upper=0.261799387798 effort=120 velocity=6.283; origin xyz=0.0715192 0 0.195982 rpy=0 0 0 -> xyz=0.1115 0 0.195982 rpy=0 0 0
- joint WaistSag: limit lower=-0.349065850398 upper=1.39626340159 effort=220 velocity=6.283 -> lower=-0.174532925199 upper=1.39626340159 effort=220 velocity=6.283
- joint WaistYaw: limit lower=-2.09439510239 upper=2.09439510239 effort=120 velocity=6.283 -> lower=-1.74532925199 upper=1.74532925199 effort=120 velocity=6.283
- joint center_bottom_led_frame_joint: child center_bottom_led_frame -> multisense/center_bottom_led_frame; parent head -> multisense/head
- joint center_top_led_frame_joint: child center_top_led_frame -> multisense/center_top_led_frame; parent head -> multisense/head
- joint gaze_joint: parent head -> multisense/head
- joint head_hokuyo_joint: child head_hokuyo_frame -> multisense/head_hokuyo_frame; parent hokuyo_link -> multisense/hokuyo_link
- joint head_imu_joint: child head_imu_link -> multisense/head_imu_link; parent head -> multisense/head
- joint hokuyo_joint: child hokuyo_link -> multisense/hokuyo_link; parent head -> multisense/head
- joint l_handj2: origin xyz=0.011908576 -0.0021833446 -0.15361558 rpy=0 0 0 -> xyz=0 -0.0305 -0.21 rpy=0 0 0
- joint left_camera_frame_joint: child left_camera_frame -> multisense/left_camera_frame; parent head -> multisense/head
- joint left_camera_optical_frame_joint: child left_camera_optical_frame -> multisense/left_camera_optical_frame; parent left_camera_frame -> multisense/left_camera_frame
- joint left_led_frame_joint: child left_led_frame -> multisense/left_led_frame; parent head -> multisense/head
- joint neck_joint: child head -> multisense/head
- joint r_handj2: origin xyz=0.011908576 0.0021833446 -0.15361558 rpy=0 0 0 -> xyz=0 0.0305 -0.21 rpy=0 0 0
- joint right_camera_frame_joint: child right_camera_frame -> multisense/right_camera_frame; parent head -> multisense/head
- joint right_camera_optical_frame_joint: child right_camera_optical_frame -> multisense/right_camera_optical_frame; parent right_camera_frame -> multisense/right_camera_frame
- joint right_led_frame_joint: child right_led_frame -> multisense/right_led_frame; parent head -> multisense/head
