Commit message: Fixed test failure

File: tests/robots/bigman/bigman.urdf (robot description, URDF)
Before this commit: robot bigman, 74 links, 73 joints
Links:
- added link imu_link2, mass 0.01; visual box size=0.01 0.01 0.01
- link DWYTorso: mass 7.31313212 -> 26
- link LFoot: mass 3.33109981 -> 3.42638110; geometry collision box size=0.32 0.16 0.015; visual mesh filename=package://bigman_urdf/meshes/NewFoot.STL scale=0.001 -0.001 0.001
- link RFoot: mass 3.33109981 -> 3.42638110; geometry collision box size=0.32 0.16 0.015; visual mesh filename=package://bigman_urdf/meshes/NewFoot.STL scale=0.001 0.001 0.001
Joints:
- added joint imu_joint2: type fixed, parent imu_link, child imu_link2, origin xyz=0 0 0.01 rpy=0 0 0
- joint LShLat: limit lower=0.0872664625995 upper=2.96705972838 effort=120 velocity=6.283 -> lower=0.0872664625995 upper=3.8571776469 effort=120 velocity=6.283
- joint LShSag: limit lower=-0.994837673634 upper=1.55334303427 effort=120 velocity=6.283 -> lower=-2.87979326578 upper=2.79252680318 effort=120 velocity=6.283
- joint NeckPitchj: limit lower=-0.436332312998 upper=1.04719755119 effort=120 velocity=6.283 -> lower=-0.261799387798 upper=1.04719755119 effort=120 velocity=6.283
- joint NeckYawj: limit lower=-3.05432619098 upper=3.05432619098 effort=120 velocity=6.283 -> lower=-0.610865238196 upper=0.610865238196 effort=120 velocity=6.283
- joint RShLat: limit lower=-2.96705972838 upper=-0.122173047639 effort=120 velocity=6.283 -> lower=-3.8571776469 upper=-0.122173047639 effort=120 velocity=6.283
- joint RShSag: limit lower=-0.994837673634 upper=1.55334303427 effort=120 velocity=6.283 -> lower=-2.84488668074 upper=2.8099800957 effort=120 velocity=6.283
- joint WaistLat: limit lower=-0.261799387798 upper=0.261799387798 effort=120 velocity=6.283 -> lower=-0.610865238196 upper=0.610865238196 effort=120 velocity=6.283
- joint WaistSag: limit lower=-0.174532925199 upper=1.39626340159 effort=220 velocity=6.283 -> lower=-0.349065850398 upper=1.39626340159 effort=220 velocity=6.283
- joint WaistYaw: limit lower=-1.74532925199 upper=1.74532925199 effort=120 velocity=6.283 -> lower=-2.84488668074 upper=2.84488668074 effort=120 velocity=6.283
- joint l_foot_lower_left_joint: origin xyz=-0.111 0.09 0 rpy=0 0 0 -> xyz=-0.16 0.09 0 rpy=0 0 0
- joint l_foot_lower_right_joint: origin xyz=-0.111 -0.07 0 rpy=0 0 0 -> xyz=-0.16 -0.07 0 rpy=0 0 0
- joint l_foot_upper_left_joint: origin xyz=0.195 0.09 0 rpy=0 0 0 -> xyz=0.16 0.09 0 rpy=0 0 0
- joint l_foot_upper_right_joint: origin xyz=0.195 -0.07 0 rpy=0 0 0 -> xyz=0.16 -0.07 0 rpy=0 0 0
- joint l_toe_joint: origin xyz=0.195 0 0 rpy=0 0 0 -> xyz=0.16 0 0 rpy=0 0 0
- joint r_foot_lower_left_joint: origin xyz=-0.111 -0.09 0 rpy=0 0 0 -> xyz=-0.16 -0.09 0 rpy=0 0 0
- joint r_foot_lower_right_joint: origin xyz=-0.111 0.07 0 rpy=0 0 0 -> xyz=-0.16 0.07 0 rpy=0 0 0
- joint r_foot_upper_left_joint: origin xyz=0.195 -0.09 0 rpy=0 0 0 -> xyz=0.16 -0.09 0 rpy=0 0 0
- joint r_foot_upper_right_joint: origin xyz=0.195 0.07 0 rpy=0 0 0 -> xyz=0.16 0.07 0 rpy=0 0 0
- joint r_toe_joint: origin xyz=0.195 0 0 rpy=0 0 0 -> xyz=0.16 0 0 rpy=0 0 0

File: tests/robots/coman/coman.urdf (robot description, URDF)
Before this commit: robot coman, 62 links, 61 joints
Links:
- removed link Xtion_body
- removed link Xtion_cam_body
- added link l_arm_ft
- added link r_arm_ft
- link DWL: geometry collision mesh filename=package://coman_urdf/meshes/simple/Torso1.STL scale=0.03937 0.03937 0.03937; visual mesh filename=package://coman_urdf/meshes/Torso1.STL scale=0.03937 0.03937 0.03937
- link DWS: geometry collision mesh filename=package://coman_urdf/meshes/simple/Torso2.STL scale=0.03937 0.03937 0.03937; visual mesh filename=package://coman_urdf/meshes/Torso2.STL scale=0.03937 0.03937 0.03937
- link DWYTorso: geometry collision mesh filename=package://coman_urdf/meshes/simple/Torso3.STL scale=0.03937 0.03937 0.03937; visual mesh filename=package://coman_urdf/meshes/Torso3.STL scale=0.03937 0.03937 0.03937
- link LElb: geometry collision mesh filename=package://coman_urdf/meshes/simple/Elbow.STL scale=1.0 1.0 1.0; visual mesh filename=package://coman_urdf/meshes/Elbow.STL scale=1.0 1.0 1.0
- link LFootmot: geometry collision mesh filename=package://coman_urdf/meshes/simple/Leg4.STL scale=0.03937 -0.03937 0.03937; visual mesh filename=package://coman_urdf/meshes/Leg4.STL scale=0.03937 -0.03937 0.03937
- link LForearm: geometry collision mesh filename=package://coman_urdf/meshes/simple/Forearm0.STL scale=1.0 1.0 1.0; visual mesh filename=package://coman_urdf/meshes/Forearm0.STL scale=0.1 0.1 0.1
- link LHipMot: geometry collision mesh filename=package://coman_urdf/meshes/simple/Leg0.STL scale=0.03937 -0.03937 0.03937; visual mesh filename=package://coman_urdf/meshes/Leg0.STL scale=0.03937 -0.03937 0.03937
- link LLowLeg: geometry collision mesh filename=package://coman_urdf/meshes/simple/Leg3.STL scale=0.03937 -0.03937 0.03937; visual mesh filename=package://coman_urdf/meshes/Leg3.STL scale=0.03937 -0.03937 0.03937
- link LShp: geometry collision mesh filename=package://coman_urdf/meshes/simple/Arm0.STL scale=0.03937 -0.03937 0.03937; visual mesh filename=package://coman_urdf/meshes/Arm0.STL scale=0.03937 -0.03937 0.03937
- link LShr: geometry collision mesh filename=package://coman_urdf/meshes/simple/Arm1.STL scale=0.03937 -0.03937 0.03937; visual mesh filename=package://coman_urdf/meshes/Arm1.STL scale=0.03937 -0.03937 0.03937
- link LShy: geometry collision mesh filename=package://coman_urdf/meshes/simple/Arm2.STL scale=0.03937 -0.03937 0.03937; visual mesh filename=package://coman_urdf/meshes/Arm2.STL scale=0.03937 -0.03937 0.03937
- link LSoftHand: geometry collision mesh filename=package://coman_urdf/meshes/simple/SoftHandOpen.STL scale=-1E-3 1E-3 1E-3; visual mesh filename=package://coman_urdf/meshes/SoftHandOpen.STL scale=-0.1 0.1 0.1
- link LThighLowLeg: geometry collision mesh filename=package://coman_urdf/meshes/simple/Leg2.STL scale=0.03937 -0.03937 0.03937; visual mesh filename=package://coman_urdf/meshes/Leg2.STL scale=0.03937 -0.03937 0.03937
- link LThighUpLeg: geometry collision mesh filename=package://coman_urdf/meshes/simple/Leg1.STL scale=0.03937 -0.03937 0.03937; visual mesh filename=package://coman_urdf/meshes/Leg1.STL scale=0.03937 -0.03937 0.03937
- link LWrMot2: geometry collision mesh filename=package://coman_urdf/meshes/simple/Forearm1.STL scale=0.001 0.001 0.001; visual mesh filename=package://coman_urdf/meshes/Forearm1.STL scale=0.001 0.001 0.001
- link LWrMot3: geometry collision mesh filename=package://coman_urdf/meshes/simple/Forearm2.STL scale=0.001 0.001 0.001; visual mesh filename=package://coman_urdf/meshes/Forearm2.STL scale=0.001 0.001 0.001
- link RElb: geometry collision mesh filename=package://coman_urdf/meshes/simple/Elbow.STL scale=1.0 1.0 1.0; visual mesh filename=package://coman_urdf/meshes/Elbow.STL scale=1.0 1.0 1.0
- link RFootmot: geometry collision mesh filename=package://coman_urdf/meshes/simple/Leg4.STL scale=0.03937 0.03937 0.03937; visual mesh filename=package://coman_urdf/meshes/Leg4.STL scale=0.03937 0.03937 0.03937
- link RForearm: geometry collision mesh filename=package://coman_urdf/meshes/simple/Forearm0.STL scale=1.0 1.0 1.0; visual mesh filename=package://coman_urdf/meshes/Forearm0.STL scale=0.1 0.1 0.1
- link RHipMot: geometry collision mesh filename=package://coman_urdf/meshes/simple/Leg0.STL scale=0.03937 0.03937 0.03937; visual mesh filename=package://coman_urdf/meshes/Leg0.STL scale=0.03937 0.03937 0.03937
- link RLowLeg: geometry collision mesh filename=package://coman_urdf/meshes/simple/Leg3.STL scale=0.03937 0.03937 0.03937; visual mesh filename=package://coman_urdf/meshes/Leg3.STL scale=0.03937 0.03937 0.03937
- link RShp: geometry collision mesh filename=package://coman_urdf/meshes/simple/Arm0.STL scale=0.03937 0.03937 0.03937; visual mesh filename=package://coman_urdf/meshes/Arm0.STL scale=0.03937 0.03937 0.03937
- link RShr: geometry collision mesh filename=package://coman_urdf/meshes/simple/Arm1.STL scale=0.03937 0.03937 0.03937; visual mesh filename=package://coman_urdf/meshes/Arm1.STL scale=0.03937 0.03937 0.03937
- link RShy: geometry collision mesh filename=package://coman_urdf/meshes/simple/Arm2.STL scale=0.03937 0.03937 0.03937; visual mesh filename=package://coman_urdf/meshes/Arm2.STL scale=0.03937 0.03937 0.03937
- link RSoftHand: geometry collision mesh filename=package://coman_urdf/meshes/simple/SoftHandOpen.STL scale=1E-3 1E-3 1E-3; visual mesh filename=package://coman_urdf/meshes/SoftHandOpen.STL scale=0.1 0.1 0.1
- link RThighLowLeg: geometry collision mesh filename=package://coman_urdf/meshes/simple/Leg2.STL scale=0.03937 0.03937 0.03937; visual mesh filename=package://coman_urdf/meshes/Leg2.STL scale=0.03937 0.03937 0.03937
- link RThighUpLeg: geometry collision mesh filename=package://coman_urdf/meshes/simple/Leg1.STL scale=0.03937 0.03937 0.03937; visual mesh filename=package://coman_urdf/meshes/Leg1.STL scale=0.03937 0.03937 0.03937
- link RWrMot2: geometry collision mesh filename=package://coman_urdf/meshes/simple/Forearm1.STL scale=0.001 0.001 0.001; visual mesh filename=package://coman_urdf/meshes/Forearm1.STL scale=0.001 0.001 0.001
- link RWrMot3: geometry collision mesh filename=package://coman_urdf/meshes/simple/Forearm2.STL scale=0.001 0.001 0.001; visual mesh filename=package://coman_urdf/meshes/Forearm2.STL scale=0.001 0.001 0.001
- link Waist: geometry collision mesh filename=package://coman_urdf/meshes/simple/Waist.STL scale=0.03937 0.03937 0.03937; visual mesh filename=package://coman_urdf/meshes/Waist.STL scale=0.03937 0.03937 0.03937
Joints:
- removed joint Xtion_body_joint
- removed joint Xtion_cam_body_joint
- added joint l_arm_ft_joint: type fixed, parent LForearm, child l_arm_ft, origin xyz=0 0 0 rpy=0 0 0
- added joint r_arm_ft_joint: type fixed, parent RForearm, child r_arm_ft, origin xyz=0 0 0 rpy=0 0 0
- joint gaze_joint: origin xyz=0.015 0 0.022 rpy=0 0 0 -> xyz=0 0 0.1 rpy=0 0 0; parent Xtion_cam_body -> torso
