Commit message: Added computeRealLinksFromFakeLinks function with test. Updated coman urdf and srdf.

File: tests/robots/coman/coman.urdf (robot description, URDF)
Before this commit: robot coman, 62 links, 61 joints
Links:
- added link l_leg_ft
- added link r_leg_ft
Joints:
- added joint l_leg_ft_joint: type fixed, parent LFoot, child l_leg_ft, origin xyz=0 0 -0.065 rpy=0 0 0
- added joint r_leg_ft_joint: type fixed, parent RFoot, child r_leg_ft, origin xyz=0 0 -0.065 rpy=0 0 0
